File: hardware/ecualizador.kicad_sch (KiCad schematic)
At the start: 72 parts, among them J1 Entrada de línea 3,5 mm, J2 Salida de línea 3,5 mm, J3 PAM8403, J4 TFT ILI9341 2,8" SPI, SW1 Pulsador, U1 MCP6004, U2 MCP6004, U3 MCP6004, U4 MCP6004, U5 ESP32-DevKitC V4

Commit message: Completa PCB de una cara, documentación LaTeX y demo con audio sincronizado
Parts:
- added C25: 100n, Ecualizador:UnaCara_C25, symbol Device:C
- added C26: 1000u 10V, Ecualizador:UnaCara_C26, symbol Device:C_Polarized
- added J5: NeoPixel 5V DIN GND, Ecualizador:UnaCara_J5, symbol Connector_Generic:Conn_01x03
- added J6: Entrada 5V 3A, Ecualizador:UnaCara_J6, symbol Connector_Generic:Conn_01x02
- added R31: 330, Ecualizador:UnaCara_R31, symbol Device:R
- added R32: 10k, Ecualizador:UnaCara_R32, symbol Device:R
- added U6: 74AHCT125, Ecualizador:UnaCara_U6, symbol 74xx:74AHCT125
- C1: footprint Capacitor_THT:CP_Radial_D6.3mm_P2.50mm -> Ecualizador:UnaCara_C1
- C10: footprint Capacitor_THT:CP_Radial_D5.0mm_P2.00mm -> Ecualizador:UnaCara_C10
- C11: footprint Capacitor_THT:C_Rect_L7.2mm_W3.0mm_P5.00mm_FKS2_FKP2_MKS2_MKP2 -> Ecualizador:UnaCara_C11
- C12: footprint Capacitor_THT:C_Rect_L7.2mm_W3.0mm_P5.00mm_FKS2_FKP2_MKS2_MKP2 -> Ecualizador:UnaCara_C12
- C13: footprint Capacitor_THT:C_Rect_L7.2mm_W3.0mm_P5.00mm_FKS2_FKP2_MKS2_MKP2 -> Ecualizador:UnaCara_C13
- C14: footprint Capacitor_THT:C_Rect_L7.2mm_W3.0mm_P5.00mm_FKS2_FKP2_MKS2_MKP2 -> Ecualizador:UnaCara_C14
- C15: footprint Capacitor_THT:C_Rect_L7.2mm_W3.0mm_P5.00mm_FKS2_FKP2_MKS2_MKP2 -> Ecualizador:UnaCara_C15
- C16: footprint Capacitor_THT:C_Rect_L7.2mm_W3.0mm_P5.00mm_FKS2_FKP2_MKS2_MKP2 -> Ecualizador:UnaCara_C16
- C17: footprint Capacitor_THT:C_Rect_L7.2mm_W3.0mm_P5.00mm_FKS2_FKP2_MKS2_MKP2 -> Ecualizador:UnaCara_C17
- C18: footprint Capacitor_THT:C_Rect_L7.2mm_W3.0mm_P5.00mm_FKS2_FKP2_MKS2_MKP2 -> Ecualizador:UnaCara_C18
- C19: footprint Capacitor_THT:CP_Radial_D5.0mm_P2.00mm -> Ecualizador:UnaCara_C19
- C2: footprint Capacitor_THT:C_Disc_D5.0mm_W2.5mm_P5.00mm -> Ecualizador:UnaCara_C2
- C20: footprint Capacitor_THT:C_Rect_L7.2mm_W3.0mm_P5.00mm_FKS2_FKP2_MKS2_MKP2 -> Ecualizador:UnaCara_C20
- C21: footprint Capacitor_THT:C_Rect_L7.2mm_W3.0mm_P5.00mm_FKS2_FKP2_MKS2_MKP2 -> Ecualizador:UnaCara_C21
- C22: footprint Capacitor_THT:C_Rect_L7.2mm_W3.0mm_P5.00mm_FKS2_FKP2_MKS2_MKP2 -> Ecualizador:UnaCara_C22
- C23: footprint Capacitor_THT:C_Rect_L7.2mm_W3.0mm_P5.00mm_FKS2_FKP2_MKS2_MKP2 -> Ecualizador:UnaCara_C23
- C24: footprint Capacitor_THT:C_Rect_L7.2mm_W3.0mm_P5.00mm_FKS2_FKP2_MKS2_MKP2 -> Ecualizador:UnaCara_C24
- C3: footprint Capacitor_THT:CP_Radial_D8.0mm_P3.50mm -> Ecualizador:UnaCara_C3
- C4: footprint Capacitor_THT:C_Disc_D5.0mm_W2.5mm_P5.00mm -> Ecualizador:UnaCara_C4
- C5: footprint Capacitor_THT:C_Disc_D5.0mm_W2.5mm_P5.00mm -> Ecualizador:UnaCara_C5
- C6: footprint Capacitor_THT:C_Disc_D5.0mm_W2.5mm_P5.00mm -> Ecualizador:UnaCara_C6
- C7: footprint Capacitor_THT:C_Disc_D5.0mm_W2.5mm_P5.00mm -> Ecualizador:UnaCara_C7
- C8: footprint Capacitor_THT:CP_Radial_D5.0mm_P2.00mm -> Ecualizador:UnaCara_C8
- C9: footprint Capacitor_THT:C_Rect_L7.2mm_W3.0mm_P5.00mm_FKS2_FKP2_MKS2_MKP2 -> Ecualizador:UnaCara_C9
- D1: footprint Diode_THT:D_DO-35_SOD27_P7.62mm_Horizontal -> Ecualizador:UnaCara_D1
- D2: footprint Diode_THT:D_DO-35_SOD27_P7.62mm_Horizontal -> Ecualizador:UnaCara_D2
- D3: footprint Diode_THT:D_DO-35_SOD27_P7.62mm_Horizontal -> Ecualizador:UnaCara_D3
- J1: footprint Connector_Audio:Jack_3.5mm_CUI_SJ1-3523N_Horizontal -> Ecualizador:UnaCara_J1
- J2: footprint Connector_Audio:Jack_3.5mm_CUI_SJ1-3523N_Horizontal -> Ecualizador:UnaCara_J2
- J3: footprint Connector_PinHeader_2.54mm:PinHeader_1x04_P2.54mm_Vertical -> Ecualizador:UnaCara_J3
- J4: value TFT ILI9341 2,8" SPI -> Waveshare 1.9 ST7789V2; footprint Connector_PinSocket_2.54mm:PinSocket_1x14_P2.54mm_Vertical -> Ecualizador:UnaCara_J4; symbol Connector_Generic:Conn_01x14 -> Connector_Generic:Conn_01x08
- R1: footprint Resistor_THT:R_Axial_DIN0207_L6.3mm_D2.5mm_P7.62mm_Horizontal -> Ecualizador:UnaCara_R1
- R10: footprint Resistor_THT:R_Axial_DIN0207_L6.3mm_D2.5mm_P7.62mm_Horizontal -> Ecualizador:UnaCara_R10
- R11: footprint Resistor_THT:R_Axial_DIN0207_L6.3mm_D2.5mm_P7.62mm_Horizontal -> Ecualizador:UnaCara_R11
- R12: footprint Resistor_THT:R_Axial_DIN0207_L6.3mm_D2.5mm_P7.62mm_Horizontal -> Ecualizador:UnaCara_R12
- R13: footprint Resistor_THT:R_Axial_DIN0207_L6.3mm_D2.5mm_P7.62mm_Horizontal -> Ecualizador:UnaCara_R13
- R14: footprint Resistor_THT:R_Axial_DIN0207_L6.3mm_D2.5mm_P7.62mm_Horizontal -> Ecualizador:UnaCara_R14
- R15: footprint Resistor_THT:R_Axial_DIN0207_L6.3mm_D2.5mm_P7.62mm_Horizontal -> Ecualizador:UnaCara_R15
- R16: footprint Resistor_THT:R_Axial_DIN0207_L6.3mm_D2.5mm_P7.62mm_Horizontal -> Ecualizador:UnaCara_R16
- R17: footprint Resistor_THT:R_Axial_DIN0207_L6.3mm_D2.5mm_P7.62mm_Horizontal -> Ecualizador:UnaCara_R17
- R18: footprint Resistor_THT:R_Axial_DIN0207_L6.3mm_D2.5mm_P7.62mm_Horizontal -> Ecualizador:UnaCara_R18
- R19: footprint Resistor_THT:R_Axial_DIN0207_L6.3mm_D2.5mm_P7.62mm_Horizontal -> Ecualizador:UnaCara_R19
- R2: footprint Resistor_THT:R_Axial_DIN0207_L6.3mm_D2.5mm_P7.62mm_Horizontal -> Ecualizador:UnaCara_R2
- R20: footprint Resistor_THT:R_Axial_DIN0207_L6.3mm_D2.5mm_P7.62mm_Horizontal -> Ecualizador:UnaCara_R20
- R21: footprint Resistor_THT:R_Axial_DIN0207_L6.3mm_D2.5mm_P7.62mm_Horizontal -> Ecualizador:UnaCara_R21
- R22: footprint Resistor_THT:R_Axial_DIN0207_L6.3mm_D2.5mm_P7.62mm_Horizontal -> Ecualizador:UnaCara_R22
- R23: footprint Resistor_THT:R_Axial_DIN0207_L6.3mm_D2.5mm_P7.62mm_Horizontal -> Ecualizador:UnaCara_R23
- R24: footprint Resistor_THT:R_Axial_DIN0207_L6.3mm_D2.5mm_P7.62mm_Horizontal -> Ecualizador:UnaCara_R24
- R25: footprint Resistor_THT:R_Axial_DIN0207_L6.3mm_D2.5mm_P7.62mm_Horizontal -> Ecualizador:UnaCara_R25
- R26: footprint Resistor_THT:R_Axial_DIN0207_L6.3mm_D2.5mm_P7.62mm_Horizontal -> Ecualizador:UnaCara_R26
- R27: footprint Resistor_THT:R_Axial_DIN0207_L6.3mm_D2.5mm_P7.62mm_Horizontal -> Ecualizador:UnaCara_R27
- R28: footprint Resistor_THT:R_Axial_DIN0207_L6.3mm_D2.5mm_P7.62mm_Horizontal -> Ecualizador:UnaCara_R28
- R29: footprint Resistor_THT:R_Axial_DIN0207_L6.3mm_D2.5mm_P7.62mm_Horizontal -> Ecualizador:UnaCara_R29
- R3: footprint Resistor_THT:R_Axial_DIN0207_L6.3mm_D2.5mm_P7.62mm_Horizontal -> Ecualizador:UnaCara_R3
- R30: value 10 -> 10k; footprint Resistor_THT:R_Axial_DIN0207_L6.3mm_D2.5mm_P7.62mm_Horizontal -> Ecualizador:UnaCara_R30
- R4: footprint Resistor_THT:R_Axial_DIN0207_L6.3mm_D2.5mm_P7.62mm_Horizontal -> Ecualizador:UnaCara_R4
- R5: footprint Resistor_THT:R_Axial_DIN0207_L6.3mm_D2.5mm_P7.62mm_Horizontal -> Ecualizador:UnaCara_R5
- R6: footprint Resistor_THT:R_Axial_DIN0207_L6.3mm_D2.5mm_P7.62mm_Horizontal -> Ecualizador:UnaCara_R6
- R7: footprint Resistor_THT:R_Axial_DIN0207_L6.3mm_D2.5mm_P7.62mm_Horizontal -> Ecualizador:UnaCara_R7
- R8: footprint Resistor_THT:R_Axial_DIN0207_L6.3mm_D2.5mm_P7.62mm_Horizontal -> Ecualizador:UnaCara_R8
- R9: footprint Resistor_THT:R_Axial_DIN0207_L6.3mm_D2.5mm_P7.62mm_Horizontal -> Ecualizador:UnaCara_R9
- RV1: footprint Potentiometer_THT:Potentiometer_Alps_RK09K_Single_Vertical -> Ecualizador:UnaCara_RV1
- RV2: footprint Potentiometer_THT:Potentiometer_Bourns_PTA3043_Single_Slide -> Ecualizador:UnaCara_RV2
- RV3: footprint Potentiometer_THT:Potentiometer_Bourns_PTA3043_Single_Slide -> Ecualizador:UnaCara_RV3
- RV4: footprint Potentiometer_THT:Potentiometer_Bourns_PTA3043_Single_Slide -> Ecualizador:UnaCara_RV4
- RV5: footprint Potentiometer_THT:Potentiometer_Alps_RK09K_Single_Vertical -> Ecualizador:UnaCara_RV5
- SW1: footprint Button_Switch_THT:SW_PUSH_6mm_H5mm -> Ecualizador:UnaCara_SW1
- U1: footprint Package_DIP:DIP-14_W7.62mm_Socket -> Ecualizador:UnaCara_U1
- U2: footprint Package_DIP:DIP-14_W7.62mm_Socket -> Ecualizador:UnaCara_U2
- U3: footprint Package_DIP:DIP-14_W7.62mm_Socket -> Ecualizador:UnaCara_U3
- U4: footprint Package_DIP:DIP-14_W7.62mm_Socket -> Ecualizador:UnaCara_U4
- U5: footprint Ecualizador:ESP32-DevKitC-38_Zocalo -> Ecualizador:UnaCara_U5
Connections:
- net +3V3: no longer R30.1
- net +5V: now also C25.1, C26.1, J5.1 (Pin_1), J6.1 (Pin_1), U6.10, U6.13, U6.14 (VCC), U6.4
- net GND: now also R30.2, C25.2, C26.2, J5.3 (Pin_3), J6.2 (Pin_2), R32.2, U6.1, U6.12, U6.5, U6.7 (GND), U6.9
- net TFT_CS: now also J4.5 (Pin_5); no longer J4.3 (Pin_3)
- net TFT_DC: now also J4.6 (Pin_6); no longer J4.5 (Pin_5)
- net TFT_MOSI: now also J4.3 (Pin_3); no longer J4.6 (Pin_6)
- net TFT_RST: now also J4.7 (Pin_7); no longer J4.4 (Pin_4)
- net TFT_SCK: now also J4.4 (Pin_4); no longer J4.7 (Pin_7)
- net LED_DATA: now reaches U5.9 (IO25)
- net LED_DATA: now also R32.1, U6.2
- net TFT_LED renamed TFT_BL
- net TFT_BL: now also R30.1, U5.27 (IO19); no longer R30.2
- removed net TFT_MISO: J4.9 (Pin_9), U5.27 (IO19)
- new net LED_5V: R31.1, U6.3
- new net LED_DIN: J5.2 (Pin_2), R31.2
- no-connect marks 26 -> 23
Other:
- note added: "Filtro RC R1–C1: fc ≈ 159 Hz. C4–C7: desacoplo local de los MCP6004."
- note added: "ILUMINACIÓN NEOPIXEL · 12 LED · FUENTE EXTERNA 5 V / 3 A"
- note added: "J4 (adaptador): 1 VCC, 2 GND, 3 DIN, 4 CLK, 5 CS, 6 DC, 7 RST, 8 BL. Waveshare 1,9 pulgadas. BL = GPIO19; datos LED = GPIO25. Cablear por nombre; GH1.25 no tiene este orden. ADC1 permite mantener el Wi-Fi activo."
- note added: "J6 alimenta la placa, el PAM8403 y los LED. No conectar simultáneamente VBUS del USB. J5: 1 = 5 V, 2 = DIN, 3 = GND. R31 cerca del primer LED; C26 junto a J5. U6 debe ser AHCT (umbral TTL): un 74HC125 a 5 V no garantiza reconocer 3,3 V. La tira vuelve a GND de potencia; no usar VREF como retorno."
- note removed: "J4: TFT ILI9341 2,8" (1 VCC 2 GND 3 CS 4 RST 5 DC 6 SDI 7 SCK 8 LED 9 SDO; 10–14 táctil, sin usar). SW1 cambia la vista (pull-up interno de GPIO27). Solo ADC1 (GPIO32–39): el ADC2 no funciona con Wi-Fi. GPIO36 lee VREF y el firmware la resta."
- note removed: "R1–C1: fc = 1/(2π·10 Ω·100 µF) = 159 Hz; aísla los amplificadores del ruido del ESP32."
